Commit message: Fixing scan merger data

File: tecdron_ros2_humble/robot_description/urdf/sick/sick_s300.xacro (robot description, xacro)
@@ -35,6 +35,12 @@
           </joint>
           <link name="${name}_link" />
+          <joint name="dummy_${name}_joint" type="fixed">
+               <parent link="${name}_link"/>
+               <child link="tecdron/base_footprint/${name}_sensor"/>
+               <origin xyz="0 0 0.115" rpy="0 0 0"/>
+          </joint>
+          <link name="tecdron/base_footprint/${name}_sensor" />
     <gazebo reference="${name}_link">
-          <sensor type="gpu_lidar" name="${name}_hokuyo_sensor">
+          <sensor type="gpu_lidar" name="${name}_sensor">
               <pose relative_to='${name}_link'>0 0 0 0 0 0</pose>
               <always_on>1</always_on>

File: tecdron_ros2_humble/robot_description/urdf/sick/sick_s300_gazebo.xacro (robot description, xacro)
@@ -9,4 +9,8 @@
                <render_engine>ogre2</render_engine>
           </plugin>
+          <plugin
+               filename="libignition-gazebo-scene-broadcaster-system.so"
+               name="ignition::gazebo::systems::SceneBroadcaster">
+          </plugin>
      </gazebo>
     </xacro:macro>

File: tecdron_ros2_humble/robot_description/urdf/tecdron.xacro (robot description, xacro)
@@ -44,5 +44,5 @@
 	</xacro:sensor_sick_s300>
 	<xacro:sensor_sick_s300 name="rear_sick" parent="base_link" color="white">
-		<origin xyz="-0.635 -0.406 0.145" rpy="${PI} 0 -${(3*PI)/4}"/>
+		<origin xyz="-0.576 -0.406 0.145" rpy="${PI} 0 -${(3*PI)/4}"/>
 	</xacro:sensor_sick_s300>
 </robot>
