Commit message: Gazebo World

File: tecdron_ros2_humble/robot_description/urdf/wheels/omni_wheel.xacro (robot description, xacro)
@@ -13,5 +13,5 @@
   </xacro:macro>
   <!-- Set up of the Wheel -->
-  <xacro:macro name="omni_wheel" params="prefix parent *origin">
+  <xacro:macro name="omni_wheel" params="prefix parent *origin ">
     <xacro:if value="${prefix == 'tecdron_front_left'}">
       <xacro:property name="fdir" value="1 -1 0" />
@@ -46,6 +46,6 @@
     </link>
     <joint name="${prefix}_wheel_joint" type="continuous">
-      <!--parent link="${parent}"/-->
-      <parent link="base_link"/>
+      <parent link="${parent}"/>
+      <!--parent link="base_link"/-->
       <child link="${prefix}_wheel_link"/>
       <xacro:insert_block name="origin" />
