Commit message: Docker Dev

File: tecdron_ros2_humble/robot_description/urdf/base/tecdron_base.xacro (robot description, xacro)
@@ -8,10 +8,9 @@
     <xacro:property name="wheel_width" value="0.175" />
     <xacro:property name="wheel_radius" value="0.127" />
-    <!-- BASE FOOTPRINT -->
+    <!-- BASE FOOTPRINT-->
     <link name="base_footprint">
       <inertial>
         <mass value="1.0" />
         <origin xyz="0 0 0" />
-        <inertia ixx="1.391" ixy="0.004" ixz="0.0" iyy="6.853" iyz="0.0" izz="10.125" />
       </inertial>
       <visual>
@@ -27,5 +26,4 @@
       <child link="base_link" />
     </joint>
-  </xacro:macro>
   <!-- BASE_LINK -->
   <link name="base_link">
@@ -37,7 +35,7 @@
     </collision>
     <inertial>
-      <mass value="100.0" />
-      <origin xyz="0 0 0" />
-      <inertia ixx="1.391" ixy="0.004" ixz="0.0" iyy="6.853" iyz="0.0" izz="10.125" />
+      <mass value="10" />
+      <origin xyz="0 0 0" rpy="0 0 0" />
+      <inertia ixx="1.5417" ixy="0" ixz="0" iyy="3.467" iyz="0" izz="4.742" />
     </inertial>
     <visual>
@@ -48,3 +46,4 @@
     </visual>
   </link>
+  </xacro:macro>
 </robot>

File: tecdron_ros2_humble/robot_description/urdf/base/tecdron_base_gazebo.xacro (robot description, xacro)
@@ -5,5 +5,5 @@
   <ros2_control name="wheel_controllers" type="system">
     <hardware>
-      <plugin>gazebo_ros2_control/GazeboSystem</plugin>
+      <plugin>ign_ros2_control/IgnitionSystem</plugin>
     </hardware>
     <joint name="tecdron_front_left_wheel_joint">
@@ -80,27 +80,14 @@
     </joint>
   </ros2_control>
-  <!-- Gazebo ros2_control plugin -->
+  <!-- Joint states plugin -->
+  <gazebo>
+    <plugin filename="ignition-gazebo-joint-state-publisher-system" name="ignition::gazebo::systems::JointStatePublisher"/>
+  </gazebo>
+    <!-- Gazebo ros2_control plugin -->
     <gazebo>
-    <plugin filename="libgazebo_ros2_control.so" name="gazebo_ros2_control">
-      <robot_sim_type>gazebo_ros2_control/GazeboSystem</robot_sim_type>
+    <plugin filename="ign_ros2_control-system" name="ign_ros2_control::IgnitionROS2ControlPlugin">
       <parameters>$(find robot_description)/config/wheel_controllers.yaml</parameters>
-    </plugin>
-  </gazebo>
-  <!-- JOINT PUBLISHER -->
-  <gazebo>
-    <plugin name="robot_joint_state" filename="libgazebo_ros_joint_state_publisher.so">
-      <ros>
-          <remapping>~/out:=joint_states</remapping>
-      </ros>
-      <update_rate>30</update_rate>
-      _visual_joint
-      <joint_name>tecdron_front_left_wheel_joint</joint_name>
-      <joint_name>tecdron_front_right_wheel_joint</joint_name>
-      <joint_name>tecdron_back_left_wheel_joint</joint_name>
-      <joint_name>tecdron_back_right_wheel_joint</joint_name>
-      <joint_name>tecdron_front_left_wheel_visual_joint</joint_name>
-      <joint_name>tecdron_front_right_wheel_visual_joint</joint_name>
-      <joint_name>tecdron_back_left_wheel_visual_joint</joint_name>
-      <joint_name>tecdron_back_right_wheel_visual_joint</joint_name>
+      <robot_param>robot_description</robot_param>
+      <robot_param_node>robot_state_publisher_node</robot_param_node>
     </plugin>
   </gazebo>

File: tecdron_ros2_humble/robot_description/urdf/sick/sick_s300.xacro (robot description, xacro)
@@ -35,41 +35,33 @@
           </joint>
           <link name="${name}_link" />
-          <!-- Sick sensor sensor for simulation -->
-         <gazebo reference="${name}_link">
-               <sensor type="ray" name="${name}_sensor">
-                    <pose>0 0 0 0 0 0</pose>
-                    <visualize>true</visualize>
-                    <update_rate>12.5</update_rate>
-                    <ray>
-                         <scan>
-                              <horizontal>
-                                   <samples>541</samples>
-                                   <resolution>1</resolution>
-                                   <min_angle>-2.20</min_angle>
-                                   <max_angle>2.3562</max_angle>-
-                              </horizontal>
-                         </scan>
-                         <range>
-                              <min>0.10</min>
-                              <max>10.0</max>
-                              <resolution>0.03</resolution>
-                         </range>
-                         <noise>
-                              <type>gaussian</type>
-                              <mean>0.0</mean>
-                              <stddev>0.03</stddev>
-                         </noise>
-                    </ray>
-                    <plugin name="${name}_laser" filename="libgazebo_ros_ray_sensor.so">
-                         <ros>
-                              <namespace></namespace>
-                              <remapping>~/out:=${name}/scan</remapping>
-                         </ros>
-                         <output_type>sensor_msgs/LaserScan</output_type>
-                         <!--topicName>${name}/scan</topicName>
-                         <frameName>/${name}_link</frameName-->
-                    </plugin>
-               </sensor>
-          </gazebo>
-     </xacro:macro>
+    <gazebo reference="${name}_link">
+          <sensor type="gpu_lidar" name="${name}_hokuyo_sensor">
+              <pose relative_to='${name}_link'>0 0 0 0 0 0</pose>
+              <always_on>1</always_on>
+              <visualize>true</visualize>
+              <update_rate>20</update_rate>
+              <topic>/${name}/laser/scan</topic>
+              <ray>
+                  <scan>
+                      <horizontal>
+                          <samples>720</samples>
+                          <resolution>1</resolution>
+                          <min_angle>${-3.1415 * (3 / 4.5)}</min_angle>
+                          <max_angle>${3.1415 * (3 / 4.5)}</max_angle>
+                      </horizontal>
+                  </scan>
+                  <range>
+                      <min>0.20</min>
+                      <max>10.0</max>
+                      <resolution>0.01</resolution>
+                  </range>
+                  <noise>
+                      <type>gaussian</type>
+                      <mean>0.0</mean>
+                      <stddev>0.01</stddev>
+                  </noise>
+              </ray>
+          </sensor>
+     </gazebo>
+</xacro:macro>
 </robot>

File: tecdron_ros2_humble/robot_description/urdf/tecdron.xacro (robot description, xacro)
@@ -6,4 +6,5 @@
 	<xacro:include filename="$(find robot_description)/urdf/base/tecdron_base.xacro" />
 	<xacro:include filename="$(find robot_description)/urdf/sick/sick_s300.xacro" />
+	<xacro:include filename="$(find robot_description)/urdf/sick/sick_s300_gazebo.xacro" />
 	<xacro:include filename="$(find robot_description)/urdf/base/tecdron_base_gazebo.xacro" />
 	<xacro:property name="wheel_offset_x" value="0.375" />
@@ -38,4 +39,5 @@
 	</xacro:omni_wheel_visual>
 	<xacro:omni_steering/>
+	<xacro:sensor_sick_s300_gazebo/>
 	<xacro:sensor_sick_s300 name="front_sick" parent="base_link" color="white">
 		<origin xyz="0.576 0.406 0.145" rpy="${PI} 0 ${PI/4}"/>

File: tecdron_ros2_humble/robot_description/urdf/wheels/omni_wheel.xacro (robot description, xacro)
@@ -5,6 +5,6 @@
   <xacro:property name="PI" value="3.1415926535897931" />
   <xacro:property name="wheel_radius" value="0.127" />
-  <xacro:property name="wheel_height" value="0.087" />
-  <xacro:property name="wheel_mass" value="10" />
+  <xacro:property name="wheel_height" value="0.036" /><!--0.087-->
+  <xacro:property name="wheel_mass" value="10.0" />
   <!-- in kg-->
   <!-- Simple Macro to calculate inertia -->
@@ -18,12 +18,11 @@
     </xacro:if>
     <xacro:if value="${prefix == 'tecdron_front_right'}">
-      <xacro:property name="visual_rotation" value="${pi}" />
       <xacro:property name="fdir" value="1 1 0" />
     </xacro:if>
     <xacro:if value="${prefix == 'tecdron_back_right'}">
-      <xacro:property name="fdir" value="1 1 0" />
+      <xacro:property name="fdir" value="1 -1 0" />
     </xacro:if>
     <xacro:if value="${prefix == 'tecdron_back_left'}">
-      <xacro:property name="fdir" value="1 -1 0" />
+      <xacro:property name="fdir" value="1 1 0" />
     </xacro:if>
     <link name="${prefix}_wheel_link">
@@ -40,5 +39,5 @@
       </inertial>
       <visual>
-        <origin xyz="0 0 0" rpy="0 0 0" />
+        <origin xyz="0 0 0" rpy="${PI/2} 0 0" />
         <geometry>
          <sphere radius="0.001"/>
@@ -52,5 +51,5 @@
       <xacro:insert_block name="origin" />
       <axis xyz="0 1 0"/>
-      <limit effort="1.27" velocity="21.0" />
+      <limit effort="1000" velocity="21.0" />
       <dynamics damping="0.001" friction="0.001" />
     </joint>
@@ -61,5 +60,5 @@
       </joint>
     </transmission>
-  <gazebo reference="${prefix}_wheel_link">
+  <gazebo reference="${prefix}_wheel_link" xmlns:ignition="http://ignitionrobotics.org/schema">
     <collision>
       <surface>
@@ -67,11 +66,11 @@
           <ode>
             <mu>1.0</mu>
-            <mu2>0.05</mu2>
-            <fdir1>${fdir}</fdir1>
+            <mu2>0.0</mu2>
+            <fdir1 ignition:expressed_in="base_link">${fdir}</fdir1>
           </ode>
         </friction>
       </surface>
     </collision>
-	</gazebo>
+  </gazebo>
   </xacro:macro>
 </robot>

Commit message: Matlab Simulations

File: tecdron_ros2_humble/robot_description/urdf/base/tecdron_base.xacro (robot description, xacro)
@@ -6,6 +6,11 @@
     <!-- Robot mechanical and motor parameters -->
     <xacro:property name="PI" value="3.1415926535897931"/>
-    <xacro:property name="wheel_width" value="0.175" />
-    <xacro:property name="wheel_radius" value="0.127" />
+    <xacro:property name="width" value="0.50" />
+    <xacro:property name="length" value="0.70" />
+    <xacro:property name="height" value="0.20" />
+    <xacro:property name="base_mass" value="150.0" />
+    <xacro:property name="ixx" value="${(1/12.0) * base_mass * (height * height + length * length)}" />
+    <xacro:property name="iyy" value="${(1/12.0) * base_mass * (width * width + length * length)}" />
+    <xacro:property name="izz" value="${(1/12.0) * base_mass * (width * width + height * height)}" />
     <!-- BASE FOOTPRINT-->
     <link name="base_footprint">
@@ -35,7 +40,7 @@
     </collision>
     <inertial>
-      <mass value="10" />
+      <mass value="${base_mass}" />
       <origin xyz="0 0 0" rpy="0 0 0" />
-      <inertia ixx="1.5417" ixy="0" ixz="0" iyy="3.467" iyz="0" izz="4.742" />
+      <inertia ixx="${ixx}" ixy="0" ixz="0" iyy="${iyy}" iyz="0" izz="${izz}" />
     </inertial>
     <visual>

File: tecdron_ros2_humble/robot_description/urdf/wheels/omni_wheel.xacro (robot description, xacro)
@@ -5,5 +5,5 @@
   <xacro:property name="PI" value="3.1415926535897931" />
   <xacro:property name="wheel_radius" value="0.127" />
-  <xacro:property name="wheel_height" value="0.036" /><!--0.087-->
+  <xacro:property name="wheel_height" value="0.036" />
   <xacro:property name="wheel_mass" value="10.0" />
   <!-- in kg-->
@@ -66,5 +66,5 @@
           <ode>
             <mu>1.0</mu>
-            <mu2>0.0</mu2>
+            <mu2>0.03</mu2>
             <fdir1 ignition:expressed_in="base_link">${fdir}</fdir1>
           </ode>
